Commit message: adeded four wheels, changed control to rear wheel only

File: description/gazebo_control.xacro (robot description, xacro)
@@ -4,6 +4,6 @@
         <plugin name= "diff_drive" filename="libgazebo_ros_diff_drive.so">
             <!-- Wheel-->
-            <left_joint>left_wheel_joint</left_joint>
-            <right_joint>right_wheel_joint</right_joint>
+            <left_joint>back_left_wheel_joint</left_joint>
+            <right_joint>back_right_wheel_joint</right_joint>
             <wheel_separation>0.25</wheel_separation>
             <wheel_diameter>0.07</wheel_diameter>

File: description/robot_core.xacro (robot description, xacro)
@@ -2,18 +2,15 @@
 <robot xmlns:xacro="http://www.ros.org/wiki/xacro" >
     <xacro:include filename="inertial_macros.xacro"/>
-    <xacro:property name="chassis_length" value="0.335"/>
-    <xacro:property name="chassis_width" value="0.265"/>
-    <xacro:property name="chassis_height" value="0.138"/>
-    <xacro:property name="chassis_mass" value="1.0"/>
-    <xacro:property name="wheel_radius" value="0.033"/>
-    <xacro:property name="wheel_thickness" value="0.026"/>
+    <xacro:property name="chassis_length" value="0.3"/>
+    <xacro:property name="chassis_width" value="0.2"/>
+    <xacro:property name="chassis_height" value="0.1"/>
+    <xacro:property name="chassis_offset_x" value="0.15"/>
+    <xacro:property name="chassis_mass" value="0.8"/>
+    <xacro:property name="wheel_radius" value="0.035"/>
+    <xacro:property name="wheel_thickness" value="0.03"/>
     <xacro:property name="wheel_mass" value="0.05"/>
-    <xacro:property name="wheel_offset_x" value="0.226"/>
-    <xacro:property name="wheel_offset_y" value="0.1485"/>
-    <xacro:property name="wheel_offset_z" value="0.01"/>
-    <xacro:property name="caster_wheel_radius" value="0.01"/>
-    <xacro:property name="caster_wheel_mass" value="0.01"/>
-    <xacro:property name="caster_wheel_offset_x" value="0.075"/>
-    <xacro:property name="caster_wheel_offset_z" value="${wheel_offset_z - wheel_radius + caster_wheel_radius}"/>
+    <xacro:property name="wheel_offset_x" value="0.1"/>
+    <xacro:property name="wheel_offset_y" value="0.12"/>
+    <xacro:property name="wheel_offset_z" value="0.175"/>
     <material name="white">
         <color rgba="1 1 1 1" />
@@ -42,9 +39,9 @@
     <link name="base_footprint">
     </link>
-    <!-- CHASSIS LINK -->
+    <!-- CHASSIS LINK - Box -->
     <joint name="chassis_joint" type="fixed">
         <parent link="base_link"/>
         <child link="chassis"/>
-        <origin xyz="${-wheel_offset_x} 0 ${-wheel_offset_z}"/>
+        <origin xyz="${-chassis_offset_x} 0 0"/>
     </joint>
     <link name="chassis">
@@ -69,12 +66,12 @@
         <material>Gazebo/Orange</material>
     </gazebo>
-    <!-- LEFT WHEEL LINK -->
-    <joint name="left_wheel_joint" type="continuous">
+    <!-- FRONT LEFT WHEEL LINK -->
+    <joint name="front_left_wheel_joint" type="continuous">
         <parent link="base_link"/>
-        <child link="left_wheel"/>
-        <origin xyz="0 ${wheel_offset_y} 0" rpy="-${pi/2} 0 0" />
+        <child link="front_left_wheel"/>
+        <origin xyz="${wheel_offset_x} ${wheel_offset_y} 0" rpy="-${pi/2} 0 0" />
         <axis xyz="0 0 1"/>
     </joint>
-    <link name="left_wheel">
+    <link name="front_left_wheel">
         <visual>
             <geometry>
@@ -95,12 +92,38 @@
         <material>Gazebo/Blue</material>
     </gazebo>
-    <!-- RIGHT WHEEL LINK -->
-    <joint name="right_wheel_joint" type="continuous">
+    <!-- REAR LEFT WHEEL LINK -->
+    <joint name="rear_left_wheel_joint" type="continuous">
         <parent link="base_link"/>
-        <child link="right_wheel"/>
-        <origin xyz="0 ${-wheel_offset_y} 0" rpy="${pi/2} 0 0" />
+        <child link="rear_left_wheel"/>
+        <origin xyz="${-wheel_offset_x} ${wheel_offset_y} 0" rpy="-${pi/2} 0 0" />
+        <axis xyz="0 0 1"/>
+    </joint>
+    <link name="rear_left_wheel">
+        <visual>
+            <geometry>
+                <cylinder radius="${wheel_radius}" length="${wheel_thickness}"/>
+            </geometry>
+            <material name="blue"/>
+        </visual>
+        <collision>
+            <geometry>
+                <sphere radius="${wheel_radius}"/>
+            </geometry>
+        </collision>
+        <xacro:inertial_cylinder mass="${wheel_mass}" length="${wheel_thickness}" radius="${wheel_radius}">
+            <origin xyz="0 0 0" rpy="0 0 0"/>
+        </xacro:inertial_cylinder>
+    </link>
+    <gazebo reference="left_wheel">
+        <material>Gazebo/Blue</material>
+    </gazebo>
+    <!-- FRONT RIGHT WHEEL LINK -->
+    <joint name="front_right_wheel_joint" type="continuous">
+        <parent link="base_link"/>
+        <child link="front_right_wheel"/>
+        <origin xyz="${wheel_offset_x} ${-wheel_offset_y} 0" rpy="${pi/2} 0 0" />
         <axis xyz="0 0 -1"/>
     </joint>
-    <link name="right_wheel">
+    <link name="front_right_wheel">
         <visual>
             <geometry>
@@ -121,30 +144,29 @@
         <material>Gazebo/Blue</material>
     </gazebo>
-    <!-- CASTER WHEEL LINK -->
-    <joint name="caster_wheel_joint" type="fixed">
-        <parent link="chassis"/>
-        <child link="caster_wheel"/>
-        <origin xyz="${caster_wheel_offset_x} 0 ${caster_wheel_offset_z}"/>
+    <!-- BACK RIGHT WHEEL LINK -->
+    <joint name="back_right_wheel_joint" type="continuous">
+        <parent link="base_link"/>
+        <child link="back_right_wheel"/>
+        <origin xyz="${-wheel_offset_x} ${-wheel_offset_y} 0" rpy="${pi/2} 0 0" />
+        <axis xyz="0 0 -1"/>
     </joint>
-    <link name="caster_wheel">
+    <link name="back_right_wheel">
         <visual>
             <geometry>
-                <sphere radius="${caster_wheel_radius}"/>
+                <cylinder radius="${wheel_radius}" length="${wheel_thickness}"/>
             </geometry>
-            <material name="white"/>
+            <material name="blue"/>
         </visual>
         <collision>
             <geometry>
-                <sphere radius="${caster_wheel_radius}"/>
+                <sphere radius="${wheel_radius}"/>
             </geometry>
         </collision>
-        <xacro:inertial_sphere mass="${caster_wheel_mass}" radius="${caster_wheel_radius}">
+        <xacro:inertial_cylinder mass="${wheel_mass}" length="${wheel_thickness}" radius="${wheel_radius}">
             <origin xyz="0 0 0" rpy="0 0 0"/>
-        </xacro:inertial_sphere>
+        </xacro:inertial_cylinder>
     </link>
-    <gazebo reference="caster_wheel">
-        <material>Gazebo/White</material>
-        <mu1 value="0.001"/>
-        <mu2 value="0.001"/>
+    <gazebo reference="right_wheel">
+        <material>Gazebo/Blue</material>
     </gazebo>
 </robot>

Commit message: control with rear drive only - working

File: description/gazebo_control.xacro (robot description, xacro)
@@ -4,6 +4,6 @@
         <plugin name= "diff_drive" filename="libgazebo_ros_diff_drive.so">
             <!-- Wheel-->
-            <left_joint>back_left_wheel_joint</left_joint>
-            <right_joint>back_right_wheel_joint</right_joint>
+            <left_joint>rear_left_wheel_joint</left_joint>
+            <right_joint>rear_right_wheel_joint</right_joint>
             <wheel_separation>0.25</wheel_separation>
             <wheel_diameter>0.07</wheel_diameter>

File: description/robot_core.xacro (robot description, xacro)
@@ -144,12 +144,12 @@
         <material>Gazebo/Blue</material>
     </gazebo>
-    <!-- BACK RIGHT WHEEL LINK -->
-    <joint name="back_right_wheel_joint" type="continuous">
+    <!-- REAR RIGHT WHEEL LINK -->
+    <joint name="rear_right_wheel_joint" type="continuous">
         <parent link="base_link"/>
-        <child link="back_right_wheel"/>
+        <child link="rear_right_wheel"/>
         <origin xyz="${-wheel_offset_x} ${-wheel_offset_y} 0" rpy="${pi/2} 0 0" />
         <axis xyz="0 0 -1"/>
     </joint>
-    <link name="back_right_wheel">
+    <link name="rear_right_wheel">
         <visual>
             <geometry>
